File: src/device.kicad_sch (KiCad schematic)
At the start: 0 parts

Commit message: stage
Parts:
- added AE1: AANI-CH-0070, symbol Device:Antenna_Chip
- added C1: C_VBUS_BULK, symbol Device:C
- added C10: C_RESET_2n2, symbol Device:C
- added C11: 1.5pF, symbol Device:C
- added C12: 2.0pF, symbol Device:C
- added C13: 0.3pF, symbol Device:C
- added C14: 3.9pF, symbol Device:C
- added C15, C17: C_DECA_100n, symbol Device:C
- added C16: C_DECD_10n, symbol Device:C
- added C2: C_VSUP_100n, symbol Device:C
- added C3: C_VCC_BULK_10u, symbol Device:C
- added C4: C_VCC_HF_100n, symbol Device:C
- added C5: C_LIN_220p, symbol Device:C
- added C6: C_PV_20p, symbol Device:C
- added C7: C_VDD_BULK_10u, symbol Device:C
- added C8: C_VDD_2u2, symbol Device:C
- added C9: C_VDD_100n, symbol Device:C
- added C_MATCH: 5.1pF, symbol Device:C
- added D1: D_VSUP_REV, symbol Device:D
- added D2: D_VSUP_TVS, symbol Device:D
- added D3: D_LIN_ESD, symbol Device:D
- added FB1: FB_120R@100MHz, symbol Device:FerriteBead
- added J1: CN-REMO, symbol Connector_Generic:Conn_01x03
- added J2: SWD_HDR, symbol Connector_Generic:Conn_01x05
- added L1: L_DCDC_4u7, symbol Device:L
- added L2: 2.7nH, symbol Device:L
- added L3, L4: 3.5nH, symbol Device:L
- added L_MATCH: 2.2nH, symbol Device:L
- added R1: R_LIN_SER_1k, symbol Device:R
- added R2: R_PV_SER_470, symbol Device:R
- added R3: R_nINT_PULLUP_10k, symbol Device:R
- added R4: R_nRST_PULLUP_10k, symbol Device:R
- added R5: R_RESET_1k, symbol Device:R
- added TP1: TP_VBUS, symbol Connector_Generic:Conn_01x01
- added TP2: TP_VSUP, symbol Connector_Generic:Conn_01x01
- added TP3: TP_3V3, symbol Connector_Generic:Conn_01x01
- added TP4: TP_GND, symbol Connector_Generic:Conn_01x01
- added TP5: TP_LIN, symbol Connector_Generic:Conn_01x01
- added TP6: TP_RESET, symbol Connector_Generic:Conn_01x01
- added U1: TLIN14313-Q1, symbol HVAC:TLIN14313-Q1
- added U2: nRF54L10, symbol HVAC:nRF54L10_QFN40
- added X1: 32.768kHz, symbol Device:Crystal
- added X2: 32MHz, symbol Device:Crystal
Connections:
- net BUS_SIG_RAW: now also D3.1 (K), J1.2 (Pin_2), R1.2
- net GND: now also AE1.2 (PCB_Trace), C1.1, C10.1, C11.1, C12.1, C13.1, C14.1, C15.1, C16.1, C17.1, C2.1, C3.1, C4.1, C5.1, C6.1, C7.1, C8.1, C9.1, C_MATCH.1, D2.2 (A), D3.2 (A), J1.1 (Pin_1), J2.2 (Pin_2), TP4.1 (Pin_1), U1.17 (WAKE), U2.24 (P0.04/CLKOUT32K), U2.34 (P1.13/AIN6), U2.41 (VSS_EP)
- net LIN_BUS: now also C5.2, R1.1, TP5.1 (Pin_1), U1.16 (WKRQ/INH)
- net PV_SENSE: now also R2.1, U2.16 (P2.06/TRACECLK)
- net RF_ANT: now also L2.2, U2.35 (P1.14/AIN7)
- net SPI_CS: now also U1.4 (WDT/CLK), U2.6 (P1.05/AIN1)
- net SPI_MISO: now also U1.6 (WDI/SDI), U2.7 (P1.06/AIN2)
- net SPI_MOSI: now also U1.5 (nWDR/SDO), U2.9 (VDD)
- net SPI_SCK: now also U1.7 (PIN/nCS), U2.10 (P2.00/SPI.DCX)
- net SWDCLK: now also J2.3 (Pin_3), U2.38 (DECD)
- net SWDIO: now also J2.4 (Pin_4), U2.39 (DCC)
- net TLIN_DIV_ON: now also U1.20 (VBAT), U2.8 (P1.08/CLK16M)
- net TLIN_nINT: now also R3.1, U1.3 (nRST), U2.1 (P1.00/XL1)
- net TLIN_nRST: now also R4.1, U1.8 (EN/nINT), U2.40 (VDD)
- net UART_RX: now also U1.18 (HSS), U2.4 (P1.03/NFC2)
- net UART_TX: now also U1.19 (LIMP), U2.3 (P1.02/NFC1)
- net VBUS_12V_RAW: now also C1.2, D1.1 (K), D2.1 (K), J1.3 (Pin_3), TP1.1 (Pin_1), U1.11 (DIV_ON)
- net VCC_3V3: now also C3.2, C4.2, FB1.2, R3.2, R4.2, TP3.1 (Pin_1), U1.9 (HSSC/FSO)
- net VDD_nRF: now also C7.2, C8.2, C9.2, FB1.1, J2.5 (Pin_5), L1.1, U2.12 (P2.02/SPI.SDO), U2.2 (P1.01/XL2), U2.21 (P0.01), U2.30 (XC2)
- net VSUP_PROT: now also C2.2, D1.2 (A), TP2.1 (Pin_1), U1.10 (PV)
- net nRF_RESET: now also J2.1 (Pin_1), R5.2, TP6.1 (Pin_1)
- new net ANT_FEED: AE1.1 (FEED), L_MATCH.1
- new net DCC: L1.2, U2.22 (SWDIO)
- new net DECA: C15.2, C17.2, U2.25 (nRESET), U2.33 (P1.12/AIN5)
- new net DECD: C16.2, U2.23 (SWDCLK)
- new net PV: C6.2, R2.2, U1.1 (VSUP)
- new net RF_50: C13.2, C14.2, C_MATCH.2, L4.1, L_MATCH.2
- new net RF_NODE1: C11.2, L2.1, L3.2
- new net RF_NODE2: C12.2, L3.1, L4.2
- new net XC1: U2.32 (P1.11/AIN4), X2.1
- new net XC2: U2.31 (VDD), X2.2
- new net XL1: U2.20 (P0.00), X1.1
- new net XL2: U2.19 (VDD), X1.2
- new net nRESET_PIN: C10.2, R5.1, U2.36 (DECA)
- no-connect marks 0 -> 17
Other:
- removed sheet 01_CN_REMO_Connector_Protection
- removed sheet 02_TLIN14313_LIN_SBC
- removed sheet 03_nRF54L10_Power_Reset_Clocks
- removed sheet 04_RF_Antenna
- removed sheet 05_Debug_Test
- note added: "CN-REMO Connector and Protection"
- note added: "Debug and Test"
- note added: "RF Network and Antenna"
- note added: "TLIN14313 LIN SBC"
- note added: "nRF54L10 Power, Reset, Clocks"

Commit message: stage
Connections:
- net DCC: now also U2.39 (DCC); no longer U2.22 (SWDIO)
- net DECA: now also U2.28 (DECRF), U2.36 (DECA); no longer U2.25 (nRESET), U2.33 (P1.12/AIN5)
- net DECD: now also U2.38 (DECD); no longer U2.23 (SWDCLK)
- net GND: now also U1.14 (GND), U2.27 (VSS_PA), U2.37 (VSS); no longer U1.17 (WAKE), U2.24 (P0.04/CLKOUT32K), U2.34 (P1.13/AIN6)
- net LIN_BUS: now also U1.15 (LIN); no longer U1.16 (WKRQ/INH)
- net PV: now also U1.10 (PV); no longer U1.1 (VSUP)
- net PV_SENSE: now also U2.5 (P1.04/AIN0); no longer U2.16 (P2.06/TRACECLK)
- net RF_ANT: now also U2.26 (ANT); no longer U2.35 (P1.14/AIN7)
- net SPI_CS: now also U1.7 (PIN/nCS), U2.15 (P2.05/SPI.CSN); no longer U1.4 (WDT/CLK), U2.6 (P1.05/AIN1)
- net SPI_MISO: now also U1.5 (nWDR/SDO), U2.14 (P2.04/SPI.SDI); no longer U1.6 (WDI/SDI), U2.7 (P1.06/AIN2)
- net SPI_MOSI: now also U1.6 (WDI/SDI), U2.12 (P2.02/SPI.SDO); no longer U1.5 (nWDR/SDO), U2.9 (VDD)
- net SPI_SCK: now also U1.4 (WDT/CLK), U2.11 (P2.01/SPI.SCK); no longer U1.7 (PIN/nCS), U2.10 (P2.00/SPI.DCX)
- net SWDCLK: now also U2.23 (SWDCLK); no longer U2.38 (DECD)
- net SWDIO: now also U2.22 (SWDIO); no longer U2.39 (DCC)
- net TLIN_DIV_ON: now also U1.11 (DIV_ON), U2.13 (P2.03); no longer U1.20 (VBAT), U2.8 (P1.08/CLK16M)
- net TLIN_nINT: now also U1.8 (EN/nINT), U2.20 (P0.00); no longer U1.3 (nRST), U2.1 (P1.00/XL1)
- net TLIN_nRST: now also U1.3 (nRST), U2.21 (P0.01); no longer U1.8 (EN/nINT), U2.40 (VDD)
- net UART_RX: now also U1.13 (RXD), U2.17 (P2.07/SWO); no longer U1.18 (HSS), U2.4 (P1.03/NFC2)
- net UART_TX: now also U1.12 (TXD), U2.18 (P2.08); no longer U1.19 (LIMP), U2.3 (P1.02/NFC1)
- net VBUS_12V_RAW: now also U1.20 (VBAT); no longer U1.11 (DIV_ON)
- net VCC_3V3: now also U1.2 (VCC); no longer U1.9 (HSSC/FSO)
- net VDD_nRF: now also U2.19 (VDD), U2.31 (VDD), U2.40 (VDD), U2.9 (VDD); no longer U2.12 (P2.02/SPI.SDO), U2.2 (P1.01/XL2), U2.21 (P0.01), U2.30 (XC2)
- net VSUP_PROT: now also U1.1 (VSUP); no longer U1.10 (PV)
- net XC1: now also U2.29 (XC1); no longer U2.32 (P1.11/AIN4)
- net XC2: now also U2.30 (XC2); no longer U2.31 (VDD)
- net XL1: now also U2.1 (P1.00/XL1); no longer U2.20 (P0.00)
- net XL2: now also U2.2 (P1.01/XL2); no longer U2.19 (VDD)
- net nRESET_PIN: now also U2.25 (nRESET); no longer U2.36 (DECA)
